File: hardware/unipad_c64/pico2w.kicad_sch (KiCad schematic)
At the start: 11 parts, among them J4 DEBUG_LA_HDR, SW1 RESET, U1 Raspberry_Pi_Pico_2_W

Commit message: board id
Parts:
- added JP1: ID0, Jumper:SolderJumper-2_P1.3mm_Open_RoundedPad1.0x1.5mm, symbol Jumper:SolderJumper_2_Open
- added JP2: ID1, Jumper:SolderJumper-2_P1.3mm_Open_RoundedPad1.0x1.5mm, symbol Jumper:SolderJumper_2_Open
- added JP3: ID2, Jumper:SolderJumper-2_P1.3mm_Open_RoundedPad1.0x1.5mm, symbol Jumper:SolderJumper_2_Open
Connections:
- net GND: now also JP1.2 (B), JP2.2 (B), JP3.2 (B)
- net BOARD_ID0: now reaches U1.31 (GPIO26_ADC0)
- net BOARD_ID0: now also JP1.1 (A)
- net BOARD_ID1: now reaches U1.32 (GPIO27_ADC1)
- net BOARD_ID1: now also JP2.1 (A)
- net BOARD_ID2: now reaches U1.34 (GPIO28_ADC2)
- net BOARD_ID2: now also JP3.1 (A)
- no-connect marks 5 -> 2
Other:
- note added: "BOARD ID STRAPPING (GP26..GP28)"
- note added: "NOTE: BOARD_ID[2:0] = {GP28, GP27, GP26} sampled once at boot via RP2350 internal pull-ups (OPEN=1, GND=0), then isolated (0 uA). Unipad C64 = 0b111 (JP1-JP3 OPEN). 3.3V-ONLY DOMAIN: GP26-GP28 (ADC0-ADC2) have an internal reverse diode to IOVDD (3.3V) — strap ONLY to GND (never 5V DB9; SYNC_1/2 use 5V FT pads GP16/GP17)."
- note removed: "NOTE: GP26-GP28 (ADC0-ADC2) are intentionally left unconnected because RP2350 ADC pads have an internal reverse diode to IOVDD (3.3V) (Pico 2 W Datasheet Section 3.2 Note, p. 13). SYNC_1/2 use 5V fail-safe FT pads GP16/GP17."
