File: hardware/unipad_c64/unipad_c64.kicad_pcb (KiCad board)
At the start: 4 copper layers, 62.5 x 60 mm, 48 parts, among them J2 PORT JOY #1, J3 PORT JOY #2, J4 DEBUG_LA_HDR, Q1 DMG2305UX, SW1 RESET, SW3 MODE, SW4 SWAP, U1 Raspberry_Pi_Pico_2_W, U4 74HCT05, U5 74HCT05, U6 74HCT05

Commit message: board id
Parts:
- added JP1: ID0, Jumper:SolderJumper-2_P1.3mm_Open_RoundedPad1.0x1.5mm, B.Cu at (122.4, 136.8)
- added JP2: ID1, Jumper:SolderJumper-2_P1.3mm_Open_RoundedPad1.0x1.5mm, B.Cu at (125.8, 136.8)
- added JP3: ID2, Jumper:SolderJumper-2_P1.3mm_Open_RoundedPad1.0x1.5mm, B.Cu at (129.2, 136.8)
Connections:
- U1 pad 31: unconnected-(U1-GPIO26_ADC0-Pad31) -> /Pico 2 W & Debug/BOARD_ID0
- U1 pad 32: unconnected-(U1-GPIO27_ADC1-Pad32) -> /Pico 2 W & Debug/BOARD_ID1
- U1 pad 34: unconnected-(U1-GPIO28_ADC2-Pad34) -> /Pico 2 W & Debug/BOARD_ID2
Routing:
- net /Pico 2 W & Debug/BOARD_ID1: track 0.00 -> 3.46 mm
- net /Pico 2 W & Debug/BOARD_ID0: track 0.00 -> 3.10 mm
- net /Pico 2 W & Debug/BOARD_ID2: track 0.00 -> 2.76 mm
Other:
- board text added: "ID0"
- board text added: "ID1"
- board text added: "ID2"
