File: hardware/unipad_c64/unipad_c64.kicad_sch (KiCad schematic)
At the start: 0 parts

Commit message: board id
Other:
- note added: "Unipad C64 - Hardware Architecture - Wireless Inputs: Bluetooth Gamepads, C64 1351 Analog Mouse, 1311/1312 Paddles & Rumble - MCU: Raspberry Pi Pico 2 W (RP2350 + CYW43439, Dual BR/EDR + BLE, PIO State Machines) - Power: <45mA from C64 +5V via 250mA PTC Polyfuse + Ferrite Pi-Filter + DMG2305UX Ideal Diode - Analog Emulation: 10k POTX/POTY pull-ups + 10k/22k (2.62V) 5V-safe SYNC dividers + 74HCT05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"
- note removed: "Unipad C64 - Hardware Architecture - Wireless Inputs: Bluetooth Gamepads, C64 1351 Analog Mouse, 1311/1312 Paddles & Rumble - MCU: Raspberry Pi Pico 2 W (RP2350 + CYW43439, Dual BR/EDR + BLE, PIO State Machines) - Power: <45mA from C64 +5V via 250mA PTC Polyfuse + Ferrite Pi-Filter + DMG2305UX Ideal Diode - Analog Emulation: 10k POTX/POTY pull-ups + 10k/22k (2.62V) 5V-safe SYNC dividers + 74HCT05"
Changed lines of the file:
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@@
 		(comment 3 "License: CC BY-NC-SA 4.0 (Attribution-NonCommercial-ShareAlike 4.0)")
 	)
-	(text "Unipad C64 - Hardware Architecture\n- Wireless Inputs: Bluetooth Gamepads, C64 1351 Analog Mouse, 1311/1312 Paddles & Rumble\n- MCU: Raspberry Pi Pico 2 W (RP2350 + CYW43439, Dual BR/EDR + BLE, PIO State Machines)\n- Power: <45mA from C64 +5V via 250mA PTC Polyfuse + Ferrite Pi-Filter + DMG2305UX Ideal Diode\n- Analog Emulation: 10k POTX/POTY pull-ups + 10k/22k (2.62V) 5V-safe SYNC dividers + 74HCT05"
+	(text "Unipad C64 - Hardware Architecture\n- Wireless Inputs: Bluetooth Gamepads, C64 1351 Analog Mouse, 1311/1312 Paddles & Rumble\n- MCU: Raspberry Pi Pico 2 W (RP2350 + CYW43439, Dual BR/EDR + BLE, PIO State Machines)\n- Power: <45mA from C64 +5V via 250mA PTC Polyfuse + Ferrite Pi-Filter + DMG2305UX Ideal Diode\n- Analog Emulation: 10k POTX/POTY pull-ups + 10k/22k (2.62V) 5V-safe SYNC dividers + 74HCT05\n- Board ID: GP26-GP28 3.3V-only bootstrap jumpers JP1-JP3 (OPEN=1, GND=0; 0b111 = Unipad C64)"
 		(exclude_from_sim no)
 		(at 62.23 48.26 0)
